File: projects/demo_project/demo_project.kicad_pcb (KiCad board)
At the start: 2 copper layers, 58.4 x 31.1 mm, 6 parts, among them J1 Screw_Terminal_01x02

Commit message: day one summary
Parts:
- added REF**: MountingHole_8.4mm_M8_Pad_Via, MountingHole:MountingHole_8.4mm_M8_Pad_Via, F.Cu at (29.9, 45.7)
- added REF**: MountingHole_8.4mm_M8_Pad_Via, MountingHole:MountingHole_8.4mm_M8_Pad_Via, F.Cu at (129.5, 45.1)
- added REF**: MountingHole_8.4mm_M8_Pad_Via, MountingHole:MountingHole_8.4mm_M8_Pad_Via, F.Cu at (130.8, 100.3)
- added REF**: MountingHole_8.4mm_M8_Pad_Via, MountingHole:MountingHole_8.4mm_M8_Pad_Via, F.Cu at (27.3, 99.7)
- moved D1 41.6 mm to (88.9, 62.2)
- moved J1 41.6 mm to (64.8, 73.9)
- moved R1 41.6 mm to (81.3, 67.9)
- moved R2 41.6 mm to (78.7, 76.2)
- moved C1 41.6 mm to (83.0, 62.2)
- moved D2 41.6 mm to (94.6, 62.2)
Routing:
- net GND: vias 0 -> 3
- added copper zone on F.Cu, net VCC
Other:
- board size 58.4 x 31.1 mm -> 125.1 x 78.7 mm
